Commit message: test urdf

File: data/urdf/franka_lnd.urdf (robot description, URDF)
Before this commit: robot franka_lnd, 17 links, 16 joints
Links:
- link main_insertion_link: geometry collision mesh filename=package://meshes/obj/tool_main_insertion_link_collision_0.t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; collision mesh filename=package://meshes/obj/tool_main_insertion_link_collision_1.o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

Commit message: pushing decimated meshes for collision

File: data/urdf/franka_lnd.urdf (robot description, URDF)
Before this commit: robot franka_lnd, 17 links, 16 joints
Links:
- link main_insertion_link: geometry collision mesh filename=package://meshes/obj/tool_main_insertion_link_collision_0.t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; collision mesh filename=package://meshes/obj/tool_main_insertion_link_collision_1.t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
- link tool_gripper1_link: geometry collision mesh filename=package://meshes/obj/lnd_gripper_link_collision_0.test.obj; collision mesh filename=package://meshes/obj/lnd_gripper_link_collision_1.test.obj
- link tool_gripper2_link: geometry collision mesh filename=package://meshes/obj/lnd_gripper_link_collision_0.test.obj; collision mesh filename=package://meshes/obj/lnd_gripper_link_collision_1.test.obj
- link tool_pitch_link: geometry collision mesh filename=package://meshes/obj/lnd_pitch_link_collision_0.test.obj; collision mesh filename=package://meshes/obj/lnd_pitch_link_collision_1.test.obj
- link tool_roll_link: geometry collision mesh filename=package://meshes/obj/lnd_roll_link_collision_0.test.obj; collision mesh filename=package://meshes/obj/lnd_roll_link_collision_1.test.obj
